File: prog-breakout/prog-breakout.kicad_pcb (KiCad board)
At the start: 2 copper layers, 29 x 17.5 mm, 4 parts, among them J1 Conn_02x05_Odd_Even, J2 Conn_01x06_Female, SW1 RESET

Commit message: Added gld logo to bottom side
Parts:
- added G***: LOGO, gld:gld-logo, B.Cu at (116.5, 80.0)
Other:
- net class Default removed
- board text added: "VCC SWCLK GND SWDIO nRST SWO"
- board text added: "prog-breakout rev B"
- board text removed: "CC BY-SA 4.0"
- board text removed: "VTARGET SWCLK GND SWDIO nRST SWO"
- board text removed: "github.com/stephendpmurphy"
- board text removed: "nucleo-stlink-adapter"
- board text removed: "rev-1"
