File: prog-breakout/prog-breakout.kicad_sch (KiCad schematic)
At the start: 4 parts, among them J1 Conn_02x05_Odd_Even, J2 Conn_01x06_Female, SW1 RESET

Commit message: Added gld logo to bottom side
Other:
- company: (none) -> greatlakesdev
- title: nucleo-stlink-adapter -> prog-breakout
Changed lines of the file:
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@@
   (paper "A4")
   (title_block
-    (title "nucleo-stlink-adapter")
-    (date "2020-08-21")
-    (rev "1")
+    (title "prog-breakout")
+    (date "2022-12-30")
+    (rev "B")
+    (company "greatlakesdev")
+    (comment 1 "CC-BY-SA")
   )
   (junction (at 110.49 90.17) (diameter 0) (color 0 0 0 0)
